File: Vanguard.kicad_pcb (KiCad board)
At the start: 4 copper layers, 55.9 x 30.5 mm, 82 parts, among them IC1 ST1L05CPU33R, IC2 MAX-M10S-00B, IC3 ADXL375BCCZ-RL, IC4 ASM330LHHTR, J1 Conn_01x02_Pin, J2 Conn_01x05_Pin, J3 MEM2067-02-180-00-A, J4 Conn_01x04_Pin, J5 Conn_01x02_Pin, J6 Screw_Terminal_01x04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

Commit message: Fixed major sensor connection error, ADXL still requires investigation
Connections:
- U5 pad 2: unconnected-(U5-CS_XL-Pad2) -> +3.3V
- U5 pad 3: unconnected-(U5-CS_MAG-Pad3) -> +3.3V
Routing:
- net GND: track 88.4 -> 91.9 mm, vias 67 -> 76
- net +3.3V: track 105.0 -> 108.2 mm, vias 16 -> 17
- net I2C1_SCL: track 91.6 -> 92.5 mm
